File: VisionCore-FPGA/FPGA.kicad_sch (KiCad schematic)
At the start: 0 parts

Commit message: Updated the PinList spreadsheet and added a GNS block and DDR block for FPGA
Other:
- added sheet PS FPGA (PS_FPGA.kicad_sch)
