File: VisionCore-FPGA/VisionCore-FPGA.kicad_pcb (KiCad board)
At the start: 2 copper layers, 1 part, among them U1 XCZU4EV-1SFVC784E

Commit message: Added some net color filtering
Parts:
- U1: value XCZU4EV-1SFVC784E -> Zynq 7000 - XCZU4EV
- moved U1 39.0 mm to (108.3, 79.7)
Connections:
- U1 pad A23: (no net) -> Net-(U1A-PS_MGTRAVTT-PadA23)
- U1 pad AA15: (no net) -> Net-(C18-Pad1)
- U1 pad AA16: (no net) -> Net-(C18-Pad1)
- U1 pad AA17: (no net) -> Net-(C18-Pad1)
- U1 pad AA18: (no net) -> Net-(C18-Pad1)
- U1 pad AA20: (no net) -> Net-(U1A-VCC_PSINTFP_DDR-PadAA20)
- U1 pad AA21: (no net) -> Net-(U1A-VCC_PSINTFP_DDR-PadAA20)
- U1 pad AB16: (no net) -> Net-(C18-Pad1)
- U1 pad B22: (no net) -> Net-(U1A-PS_MGTRAVCC-PadB22)
- U1 pad C23: (no net) -> Net-(U1A-PS_MGTRAVTT-PadA23)
- U1 pad D22: (no net) -> Net-(U1A-PS_MGTRAVCC-PadB22)
- U1 pad D25: (no net) -> Net-(U1A-PS_MGTRAVTT-PadA23)
- U1 pad E23: (no net) -> Net-(U1A-PS_MGTRAVTT-PadA23)
- U1 pad K10: (no net) -> Net-(C1-Pad1)
- U1 pad L10: (no net) -> Net-(C1-Pad1)
- U1 pad L11: (no net) -> Net-(C15-Pad1)
- U1 pad L12: (no net) -> Net-(C15-Pad1)
- U1 pad M10: (no net) -> Net-(C1-Pad1)
- U1 pad M11: (no net) -> Net-(C15-Pad1)
- U1 pad M12: (no net) -> Net-(C15-Pad1)
- U1 pad M13: (no net) -> Net-(C26-Pad1)
- U1 pad M14: (no net) -> Net-(C26-Pad1)
- U1 pad M15: (no net) -> Net-(C26-Pad1)
- U1 pad M16: (no net) -> Net-(C26-Pad1)
- U1 pad M9: (no net) -> Net-(C1-Pad1)
- U1 pad N11: (no net) -> Net-(C1-Pad1)
- U1 pad N13: (no net) -> Net-(C1-Pad1)
- U1 pad N15: (no net) -> Net-(C1-Pad1)
- U1 pad N16: (no net) -> Net-(C26-Pad1)
- U1 pad P10: (no net) -> Net-(C1-Pad1)
- U1 pad P14: (no net) -> Net-(C1-Pad1)
- U1 pad P15: (no net) -> Net-(C1-Pad1)
- U1 pad P4: (no net) -> Net-(U1A-MGTAVTT_R-PadP4)
- U1 pad R10: (no net) -> Net-(C1-Pad1)
- U1 pad R11: (no net) -> Net-(C1-Pad1)
- U1 pad R14: (no net) -> Net-(C1-Pad1)
- U1 pad T11: (no net) -> Net-(C1-Pad1)
- U1 pad T15: (no net) -> Net-(C1-Pad1)
- U1 pad T16: (no net) -> Net-(U1A-VCC_PSPLL-PadT16)
- U1 pad T17: (no net) -> Net-(U1A-VCC_PSPLL-PadT16)
- U1 pad T18: (no net) -> Net-(U1A-VCC_PSPLL-PadT16)
- U1 pad T4: (no net) -> Net-(U1A-MGTAVTT_R-PadP4)
- U1 pad U10: (no net) -> Net-(C1-Pad1)
- U1 pad U14: (no net) -> Net-(C1-Pad1)
- U1 pad U15: (no net) -> Net-(C1-Pad1)
- U1 pad U16: (no net) -> Net-(U1A-VCC_PSDDR_PLL-PadU16)
- U1 pad U18: (no net) -> Net-(U1A-VCC_PSDDR_PLL-PadU16)
- U1 pad U19: (no net) -> Net-(C24-Pad1)
- U1 pad U20: (no net) -> Net-(C24-Pad1)
- U1 pad U21: (no net) -> Net-(U1A-VCCINT_VCU-PadU21)
- U1 pad U5: (no net) -> Net-(U1A-MGTVCCAUX_R-PadU5)
- U1 pad V10: (no net) -> Net-(C1-Pad1)
- U1 pad V11: (no net) -> Net-(C1-Pad1)
- U1 pad V12: (no net) -> Net-(C1-Pad1)
- U1 pad V14: (no net) -> Net-(C1-Pad1)
- U1 pad V16: /FPGA/TEST -> Net-(C21-Pad1)
- U1 pad V17: (no net) -> Net-(C21-Pad1)
- U1 pad V18: (no net) -> Net-(C21-Pad1)
- U1 pad V19: (no net) -> Net-(C24-Pad1)
- U1 pad V20: (no net) -> Net-(U1A-VCCINT_VCU-PadU21)
- U1 pad V21: (no net) -> Net-(U1A-VCCINT_VCU-PadU21)
- U1 pad V4: (no net) -> Net-(U1A-MGTAVCC_R-PadV4)
- U1 pad W15: (no net) -> Net-(C21-Pad1)
- U1 pad W16: (no net) -> Net-(C21-Pad1)
- U1 pad W17: (no net) -> Net-(C21-Pad1)
- U1 pad W19: (no net) -> Net-(C24-Pad1)
- U1 pad W21: (no net) -> Net-(U1A-VCCINT_VCU-PadU21)
- U1 pad W5: (no net) -> Net-(U1A-MGTVCCAUX_R-PadU5)
- U1 pad Y15: (no net) -> Net-(C18-Pad1)
- U1 pad Y17: (no net) -> Net-(C18-Pad1)
- U1 pad Y18: (no net) -> unconnected-(U1A-VCC_PSBATT-PadY18)
- U1 pad Y19: (no net) -> Net-(U1A-VCC_PSINTFP_DDR-PadAA20)
- U1 pad Y20: (no net) -> unconnected-(U1A-VCC_PSADC-PadY20)
- U1 pad Y21: (no net) -> Net-(U1A-VCCINT_VCU-PadU21)
- U1 pad Y4: (no net) -> Net-(U1A-MGTAVCC_R-PadV4)
